Commit message: fix Digit effort limits and arms

File: robots/digit_description/robots/digit-v3-armfixed-springfixed.urdf (robot description, URDF)
Before this commit: robot digit-v3-armfixed-floatingbase, 43 links, 42 joints
Joints:
- joint left_A2: limit lower=-1.7453 upper=1.7453 effort=0.9 velocity=11.5 -> lower=-1.7453 upper=1.7453 effort=0 velocity=11.5
- joint left_B2: limit lower=-1.7453 upper=1.7453 effort=0.9 velocity=11.5 -> lower=-1.7453 upper=1.7453 effort=0 velocity=11.5
- joint left_ach2: limit lower=-1.7453 upper=1.7453 effort=0.9 velocity=11.5 -> lower=-1.7453 upper=1.7453 effort=0 velocity=11.5
- joint left_achilles_rod: limit lower=-1.7453 upper=1.7453 effort=12.5 velocity=8.5085 -> lower=-1.7453 upper=1.7453 effort=0 velocity=8.5085
- joint left_elbow: limit lower=-1.3526 upper=1.3526 effort=1.4 velocity=12.5 -> lower=-1.3526 upper=1.3526 effort=113.000 velocity=12.5; origin xyz=0 -0.0385 0.185 rpy=1.5707963267948966192313216916398 -0.3926991 0 -> xyz=0 -0.0385 0.185 rpy=1.5707963267948966192313216916398 -0.3926990817 0; type fixed -> revolute
- joint left_heel_spring: limit lower=-0.1047 upper=0.1047 effort=12 velocity=11.5 -> lower=-0.1047 upper=0.1047 effort=0 velocity=11.5
- joint left_hip_pitch: limit lower=-1.0472 upper=1.5707963267948966192313216916398 effort=12.5 velocity=8.5 -> lower=-1.0472 upper=1.5707963267948966192313216916398 effort=216.928 velocity=8.5
- joint left_hip_roll: limit lower=-1.0472 upper=1.0472 effort=1.4 velocity=12.15 -> lower=-1.0472 upper=1.0472 effort=113 velocity=12.15
- joint left_hip_yaw: limit lower=-0.698132 upper=0.698132 effort=1.4 velocity=12.15 -> lower=-0.698132 upper=0.698132 effort=79.1765 velocity=12.15
- joint left_knee: limit lower=-1.3963 upper=1.0193 effort=12.5 velocity=8.5085 -> lower=-1.3963 upper=1.0193 effort=231.317 velocity=8.5085
- joint left_shoulder_pitch: limit lower=-2.5307 upper=2.5307 effort=1.4 velocity=12.5 -> lower=-2.5307 upper=2.5307 effort=113.000 velocity=12.5; origin xyz=-0.00317 -0.011055 0.0555 rpy=1.5707963267948966192313216916398 1.875658163397448285891755404009 -0.2792527 -> xyz=-0.00317 -0.011055 0.0555 rpy=1.5707963267948966192313216916398 0.7853981634 -0.2792526803; type fixed -> revolute
- joint left_shoulder_roll: limit lower=-1.309 upper=1.309 effort=1.4 velocity=12.5 -> lower=-1.309 upper=1.309 effort=113.000 velocity=12.5; origin xyz=-0.001 0.12 0.4 rpy=-1.5707963267948966192313216916398 -1.5467303 1.5707963267948966192313216916398 -> xyz=-0.001 0.12 0.4 rpy=-1.5707963267948966192313216916398 -1.396263402 1.5707963267948966192313216916398; type fixed -> revolute
- joint left_shoulder_yaw: limit lower=-1.7453 upper=1.7453 effort=1.4 velocity=10 -> lower=-1.7453 upper=1.7453 effort=79.1765 velocity=10; origin xyz=0 -0.165 -0.1 rpy=1.5707963267948966192313216916398 -0.14981736 0 -> xyz=0 -0.165 -0.1 rpy=1.5707963267948966192313216916398 0 0; type fixed -> revolute
- joint left_toe_A: limit lower=-0.8077 upper=0.7851 effort=0.9 velocity=11.5 -> lower=-0.8077 upper=0.7851 effort=41.9759 velocity=11.5
- joint left_toe_A_rod: limit lower=-1.7453 upper=1.7453 effort=0.9 velocity=11.5 -> lower=-1.7453 upper=1.7453 effort=0 velocity=11.5
- joint left_toe_B: limit lower=-0.8010 upper=0.7950 effort=0.9 velocity=11.5 -> lower=-0.8010 upper=0.7950 effort=41.9759 velocity=11.5
- joint left_toe_B_rod: limit lower=-1.7453 upper=1.7453 effort=0.9 velocity=11.5 -> lower=-1.7453 upper=1.7453 effort=0 velocity=11.5
- joint left_toe_pitch: limit lower=-0.7679 upper=0.5934 effort=0.9 velocity=11.5 -> lower=-0.7679 upper=0.5934 effort=0 velocity=11.5
- joint left_toe_roll: limit lower=-0.6458 upper=0.5760 effort=0.9 velocity=11.5 -> lower=-0.6458 upper=0.5760 effort=0 velocity=11.5
- joint right_A2: limit lower=-1.7453 upper=1.7453 effort=0.9 velocity=11.5 -> lower=-1.7453 upper=1.7453 effort=0 velocity=11.5
- joint right_B2: limit lower=-1.7453 upper=1.7453 effort=0.9 velocity=11.5 -> lower=-1.7453 upper=1.7453 effort=0 velocity=11.5
- joint right_ach2: limit lower=-1.7453 upper=1.7453 effort=0.9 velocity=11.5 -> lower=-1.7453 upper=1.7453 effort=0 velocity=11.5
- joint right_achilles_rod: limit lower=-1.7453 upper=1.7453 effort=12.5 velocity=8.5085 -> lower=-1.7453 upper=1.7453 effort=0 velocity=8.5085
- joint right_elbow: limit lower=-1.3526 upper=1.3526 effort=1.4 velocity=12.5 -> lower=-1.3526 upper=1.3526 effort=113.000 velocity=12.5; origin xyz=0 0.0385 0.185 rpy=-1.5707963267948966192313216916398 -0.3926991 0 -> xyz=0 0.0385 0.185 rpy=-1.5707963267948966192313216916398 -0.3926990817 0; type fixed -> revolute
- joint right_heel_spring: limit lower=-0.1047 upper=0.1047 effort=12 velocity=11.5 -> lower=-0.1047 upper=0.1047 effort=0 velocity=11.5
- joint right_hip_pitch: limit lower=-1.5707963267948966192313216916398 upper=1.0472 effort=12.5 velocity=8.5 -> lower=-1.5707963267948966192313216916398 upper=1.0472 effort=216.928 velocity=8.5
- joint right_hip_roll: limit lower=-1.0472 upper=1.0472 effort=1.4 velocity=12.15 -> lower=-1.0472 upper=1.0472 effort=113.000 velocity=12.15
- joint right_hip_yaw: limit lower=-0.698132 upper=0.698132 effort=1.4 velocity=12.15 -> lower=-0.698132 upper=0.698132 effort=79.1765 velocity=12.15
- joint right_knee: limit lower=-1.0193 upper=1.3963 effort=12.5 velocity=8.5085 -> lower=-1.0193 upper=1.3963 effort=231.317 velocity=8.5085
- joint right_shoulder_pitch: limit lower=-2.5307 upper=2.5307 effort=1.4 velocity=12.5 -> lower=-2.5307 upper=2.5307 effort=113.000 velocity=12.5; origin xyz=-0.00317 0.011055 0.0555 rpy=-1.5707963267948966192313216916398 1.875658163397448285891755404009 0.2792527 -> xyz=-0.00317 0.011055 0.0555 rpy=-1.5707963267948966192313216916398 0.7853981634 0.2792526803; type fixed -> revolute
- joint right_shoulder_roll: limit lower=-1.309 upper=1.309 effort=1.4 velocity=12.5 -> lower=-1.309 upper=1.309 effort=113.000 velocity=12.5; origin xyz=-0.001 -0.12 0.4 rpy=1.5707963267948966192313216916398 -1.5467303 -1.5707963267948966192313216916398 -> xyz=-0.001 -0.12 0.4 rpy=1.5707963267948966192313216916398 -1.396263402 -1.5707963267948966192313216916398; type fixed -> revolute
- joint right_shoulder_yaw: limit lower=-1.7453 upper=1.7453 effort=1.4 velocity=10 -> lower=-1.7453 upper=1.7453 effort=79.1765 velocity=10; origin xyz=0 0.165 -0.1 rpy=-1.5707963267948966192313216916398 -0.14981736 0 -> xyz=0 0.165 -0.1 rpy=-1.5707963267948966192313216916398 0 0; type fixed -> revolute
- joint right_toe_A: limit lower=-0.7851 upper=0.8077 effort=0.9 velocity=11.5 -> lower=-0.7851 upper=0.8077 effort=41.9759 velocity=11.5
- joint right_toe_A_rod: limit lower=-1.7453 upper=1.7453 effort=0.9 velocity=11.5 -> lower=-1.7453 upper=1.7453 effort=0 velocity=11.5
- joint right_toe_B: limit lower=-0.7950 upper=0.8010 effort=0.9 velocity=11.5 -> lower=-0.7950 upper=0.8010 effort=41.9759 velocity=11.5
- joint right_toe_B_rod: limit lower=-1.7453 upper=1.7453 effort=0.9 velocity=11.5 -> lower=-1.7453 upper=1.7453 effort=0 velocity=11.5
- joint right_toe_pitch: limit lower=-0.5934 upper=0.7679 effort=0.9 velocity=11.5 -> lower=-0.5934 upper=0.7679 effort=0 velocity=11.5
- joint right_toe_roll: limit lower=-0.5760 upper=0.6458 effort=0.9 velocity=11.5 -> lower=-0.5760 upper=0.6458 effort=0 velocity=11.5
