Commit message: change joint names so that they are different from link

File: robots/digit_description/robots/digit-v3-springfixed.urdf (robot description, URDF)
Before this commit: robot digit-v3-springfixed, 43 links, 42 joints
Joints:
- removed joint left_A2
- removed joint left_B2
- removed joint left_ach2
- removed joint left_achilles_rod
- removed joint left_elbow
- removed joint left_heel_spring
- removed joint left_hip_pitch
- removed joint left_hip_roll
- removed joint left_hip_yaw
- removed joint left_knee
- removed joint left_shin
- removed joint left_shoulder_pitch
- removed joint left_shoulder_roll
- removed joint left_shoulder_yaw
- removed joint left_tarsus
- removed joint left_toe_A
- removed joint left_toe_A_rod
- removed joint left_toe_B
- removed joint left_toe_B_rod
- removed joint left_toe_pitch
- removed joint left_toe_roll
- removed joint right_A2
- removed joint right_B2
- removed joint right_ach2
- removed joint right_achilles_rod
- removed joint right_elbow
- removed joint right_heel_spring
- removed joint right_hip_pitch
- removed joint right_hip_roll
- removed joint right_hip_yaw
- removed joint right_knee
- removed joint right_shin
- removed joint right_shoulder_pitch
- removed joint right_shoulder_roll
- removed joint right_shoulder_yaw
- removed joint right_tarsus
- removed joint right_toe_A
- removed joint right_toe_A_rod
- removed joint right_toe_B
- removed joint right_toe_B_rod
- removed joint right_toe_pitch
- removed joint right_toe_roll
- added joint left_A2_joint: type revolute, parent left_toe_A_rod, child left_A2, origin xyz=0 0 0 rpy=0 0 0, axis 0 1 0, limit lower=-1.7453 upper=1.7453 effort=0 velocity=11.5
- added joint left_B2_joint: type revolute, parent left_toe_B_rod, child left_B2, origin xyz=0 0 0 rpy=0 0 0, axis 0 1 0, limit lower=-1.7453 upper=1.7453 effort=0 velocity=11.5
- added joint left_ach2_joint: type revolute, parent left_achilles_rod, child left_ach2, origin xyz=0 0 0 rpy=0 0 0, axis 0 1 0, limit lower=-1.7453 upper=1.7453 effort=0 velocity=11.5
- added joint left_achilles_rod_joint: type revolute, parent left_hip_pitch, child left_achilles_rod, origin xyz=0 0 0.046 rpy=0.0087528908613780896652567520277444 0.07085157762907765000015558598534 -1.4355410054288866295024718056084, axis 0 0 1, limit lower=-1.7453 upper=1.7453 effort=0 velocity=8.5085
- added joint left_elbow_joint: type revolute, parent left_shoulder_yaw, child left_elbow, origin xyz=0 -0.0385 0.185 rpy=1.5707963267948966192313216916398 -0.3926990817 0, axis 0 0 1, limit lower=-1.3526 upper=1.3526 effort=113.000 velocity=12.5
- added joint left_heel_spring_joint: type fixed, parent left_tarsus, child left_heel_spring, origin xyz=-0.01766 -0.029456 0.00104 rpy=-0.068907263191147760661436905138544 -0.03703539652360886280657581437481 2.7207176029176958209632175567094, axis 0 0 1, limit lower=-0.1047 upper=0.1047 effort=0 velocity=11.5
- added joint left_hip_pitch_joint: type revolute, parent left_hip_yaw, child left_hip_pitch, origin xyz=0 0.004 0.068 rpy=-1.5707963267948966192313216916398 -0.78539816339739465522740147207514 3.1415926535897932384626433832795, axis 0 0 -1, limit lower=-1.0472 upper=1.5707963267948966192313216916398 effort=216.928 velocity=8.5
- added joint left_hip_roll_joint: type revolute, parent torso, child left_hip_roll, origin xyz=-0.001 0.091 0 rpy=1.5707963267948966192313216916398 -1.1955515003397312323585310878116 -1.5707963267948966192313216916398, axis 0 0 1, limit lower=-1.0472 upper=1.0472 effort=113 velocity=12.15
- added joint left_hip_yaw_joint: type revolute, parent left_hip_roll, child left_hip_yaw, origin xyz=-0.0505 0 0.044 rpy=0   -1.5707963267948966192313216916398         0, axis 0 0 1, limit lower=-0.698132 upper=0.698132 effort=79.1765 velocity=12.15
- added joint left_knee_joint: type revolute, parent left_hip_pitch, child left_knee, origin xyz=0.12 0 0.0045 rpy=0         0   -1.5707963267948966192313216916398, axis 0 0 1, limit lower=-1.3963 upper=1.0193 effort=231.317 velocity=8.5085
- added joint left_shin_joint: type fixed, parent left_knee, child left_shin, origin xyz=0.060677 0.047406 0 rpy=0 0 0, axis 0 0 1, limit lower=-0.35 upper=0.35 effort=0 velocity=10
- added joint left_shoulder_pitch_joint: type revolute, parent left_shoulder_roll, child left_shoulder_pitch, origin xyz=-0.00317 -0.011055 0.0555 rpy=1.5707963267948966192313216916398 0.7853981634 -0.2792526803, axis 0 0 -1, limit lower=-2.5307 upper=2.5307 effort=113.000 velocity=12.5
- added joint left_shoulder_roll_joint: type revolute, parent torso, child left_shoulder_roll, origin xyz=-0.001 0.12 0.4 rpy=-1.5707963267948966192313216916398 -1.396263402 1.5707963267948966192313216916398, axis 0 0 1, limit lower=-1.309 upper=1.309 effort=113.000 velocity=12.5
- added joint left_shoulder_yaw_joint: type revolute, parent left_shoulder_pitch, child left_shoulder_yaw, origin xyz=0 -0.165 -0.1 rpy=1.5707963267948966192313216916398 0 0, axis 0 0 1, limit lower=-1.7453 upper=1.7453 effort=79.1765 velocity=10
- added joint left_tarsus_joint: type revolute, parent left_shin, child left_tarsus, origin xyz=0.434759 0.02 0 rpy=0         0    1.7976883650999471164766418951331, axis 0 0 1, limit lower=-0.8779 upper=1.2497 effort=0 velocity=20
- added joint left_toe_A_joint: type revolute, parent left_tarsus, child left_toe_A, origin xyz=0.059 -0.034 -0.0276 rpy=3.1415926535897932384626433832795 0 -1.5526449025733231046331184188602, axis 0 0 1, limit lower=-0.8077 upper=0.7851 effort=41.9759 velocity=11.5
- added joint left_toe_A_rod_joint: type revolute, parent left_toe_A, child left_toe_A_rod, origin xyz=0.057 0 -0.008 rpy=-0.037175987474526640819139089444434 0.0069420091856212517295032782271846 -1.5437619437662688515189302052022, axis 0 0 1, limit lower=-1.7453 upper=1.7453 effort=0 velocity=11.5
- added joint left_toe_B_joint: type revolute, parent left_tarsus, child left_toe_B, origin xyz=0.111 -0.034 0.0276 rpy=0         0   -1.5526446425200970402613620535703, axis 0 0 1, limit lower=-0.8010 upper=0.7950 effort=41.9759 velocity=11.5
- added joint left_toe_B_rod_joint: type revolute, parent left_toe_B, child left_toe_B_rod, origin xyz=0.057 0 -0.008 rpy=-0.053844685552438438513878082858355 0.0022826832958013874852465363574083 1.5418663490001245364169335516635, axis 0 0 1, limit lower=-1.7453 upper=1.7453 effort=0 velocity=11.5
- added joint left_toe_pitch_joint: type revolute, parent left_tarsus, child left_toe_pitch, origin xyz=0.408 -0.04 0 rpy=0         0    1.2522744638393012994725950193242, axis 0 0 1, limit lower=-0.7679 upper=0.5934 effort=0 velocity=11.5
- added joint left_toe_roll_joint: type revolute, parent left_toe_pitch, child left_toe_roll, origin xyz=0 0 0 rpy=0    1.5707963267948966192313216916398         0, axis 0 0 1, limit lower=-0.6458 upper=0.5760 effort=0 velocity=11.5
- added joint right_A2_joint: type revolute, parent right_toe_A_rod, child right_A2, origin xyz=0 0 0 rpy=0 0 0, axis 0 1 0, limit lower=-1.7453 upper=1.7453 effort=0 velocity=11.5
- added joint right_B2_joint: type revolute, parent right_toe_B_rod, child right_B2, origin xyz=0 0 0 rpy=0 0 0, axis 0 1 0, limit lower=-1.7453 upper=1.7453 effort=0 velocity=11.5
- added joint right_ach2_joint: type revolute, parent right_achilles_rod, child right_ach2, origin xyz=0 0 0 rpy=0 0 0, axis 0 1 0, limit lower=-1.7453 upper=1.7453 effort=0 velocity=11.5
- added joint right_achilles_rod_joint: type revolute, parent right_hip_pitch, child right_achilles_rod, origin xyz=0 0 0.046 rpy=-0.0087523017375784415566863927438135 0.070851391807226243857442682383407 1.4355417226017064269427692124736, axis 0 0 1, limit lower=-1.7453 upper=1.7453 effort=0 velocity=8.5085
- added joint right_elbow_joint: type revolute, parent right_shoulder_yaw, child right_elbow, origin xyz=0 0.0385 0.185 rpy=-1.5707963267948966192313216916398 -0.3926990817 0, axis 0 0 1, limit lower=-1.3526 upper=1.3526 effort=113.000 velocity=12.5
- added joint right_heel_spring_joint: type fixed, parent right_tarsus, child right_heel_spring, origin xyz=-0.01766 0.029456 0.00104 rpy=0.068907849662554282454962617521232 -0.037035299439698535217679875586327 -2.7207170387858861104746210912708, axis 0 0 1, limit lower=-0.1047 upper=0.1047 effort=0 velocity=11.5
- added joint right_hip_pitch_joint: type revolute, parent right_hip_yaw, child right_hip_pitch, origin xyz=0 -0.004 0.068 rpy=1.5707963267948966192313216916398 -0.78539855435120076165844693605322 3.1415926535897932384626433832795, axis 0 0 -1, limit lower=-1.5707963267948966192313216916398 upper=1.0472 effort=216.928 velocity=8.5
- added joint right_hip_roll_joint: type revolute, parent torso, child right_hip_roll, origin xyz=-0.001 -0.091 0 rpy=-1.5707963267948966192313216916398 -1.1955515003397312323585310878116 1.5707963267948966192313216916398, axis 0 0 1, limit lower=-1.0472 upper=1.0472 effort=113.000 velocity=12.15
- added joint right_hip_yaw_joint: type revolute, parent right_hip_roll, child right_hip_yaw, origin xyz=-0.0505 0 0.044 rpy=0   -1.5707963267948966192313216916398         0, axis 0 0 1, limit lower=-0.698132 upper=0.698132 effort=79.1765 velocity=12.15
- added joint right_knee_joint: type revolute, parent right_hip_pitch, child right_knee, origin xyz=0.12 0 0.0045 rpy=0         0    1.5707963267948966192313216916398, axis 0 0 1, limit lower=-1.0193 upper=1.3963 effort=231.317 velocity=8.5085
- added joint right_shin_joint: type fixed, parent right_knee, child right_shin, origin xyz=0.060677 -0.047406 0 rpy=0 0 0, axis 0 0 1, limit lower=-0.35 upper=0.35 effort=0 velocity=10
- added joint right_shoulder_pitch_joint: type revolute, parent right_shoulder_roll, child right_shoulder_pitch, origin xyz=-0.00317 0.011055 0.0555 rpy=-1.5707963267948966192313216916398 0.7853981634 0.2792526803, axis 0 0 -1, limit lower=-2.5307 upper=2.5307 effort=113.000 velocity=12.5
- added joint right_shoulder_roll_joint: type revolute, parent torso, child right_shoulder_roll, origin xyz=-0.001 -0.12 0.4 rpy=1.5707963267948966192313216916398 -1.396263402 -1.5707963267948966192313216916398, axis 0 0 1, limit lower=-1.309 upper=1.309 effort=113.000 velocity=12.5
- added joint right_shoulder_yaw_joint: type revolute, parent right_shoulder_pitch, child right_shoulder_yaw, origin xyz=0 0.165 -0.1 rpy=-1.5707963267948966192313216916398 0 0, axis 0 0 1, limit lower=-1.7453 upper=1.7453 effort=79.1765 velocity=10
- added joint right_tarsus_joint: type revolute, parent right_shin, child right_tarsus, origin xyz=0.434759 -0.02 0 rpy=0         0   -1.7976883650999471164766418951331, axis 0 0 1, limit lower=-1.2497 upper=0.8779 effort=0 velocity=20
- added joint right_toe_A_joint: type revolute, parent right_tarsus, child right_toe_A, origin xyz=0.059 0.034 -0.0276 rpy=3.1415926535897932384626433832795 0 1.5526446425200970402613620535703, axis 0 0 1, limit lower=-0.7851 upper=0.8077 effort=41.9759 velocity=11.5
- added joint right_toe_A_rod_joint: type revolute, parent right_toe_A, child right_toe_A_rod, origin xyz=0.057 0 -0.008 rpy=0.03717647899635967423392912678537 0.0069418384185932916277672610760874 1.5437611240201540852012840332463, axis 0 0 1, limit lower=-1.7453 upper=1.7453 effort=0 velocity=11.5
- added joint right_toe_B_joint: type revolute, parent right_tarsus, child right_toe_B, origin xyz=0.111 0.034 0.0276 rpy=0         0    1.5526446425200970402613620535703, axis 0 0 1, limit lower=-0.7950 upper=0.8010 effort=41.9759 velocity=11.5
- added joint right_toe_B_rod_joint: type revolute, parent right_toe_B, child right_toe_B_rod, origin xyz=0.057 0 -0.008 rpy=0.053844685552438438513878082858355 0.0022826832958013874852465363574083 -1.5418663490001245364169335516635, axis 0 0 1, limit lower=-1.7453 upper=1.7453 effort=0 velocity=11.5
- added joint right_toe_pitch_joint: type revolute, parent right_tarsus, child right_toe_pitch, origin xyz=0.408 0.04 0 rpy=0         0   -1.2522744638393012994725950193242, axis 0 0 1, limit lower=-0.5934 upper=0.7679 effort=0 velocity=11.5
- added joint right_toe_roll_joint: type revolute, parent right_toe_pitch, child right_toe_roll, origin xyz=0 0 0 rpy=0    1.5707963267948966192313216916398         0, axis 0 0 1, limit lower=-0.5760 upper=0.6458 effort=0 velocity=11.5
